File: ergogen/pcbs/left.kicad_pcb (KiCad board)
At the start: 2 copper layers, 167 x 141 mm, 62 parts

Commit message: decided to go reversible pcb route, removed right side and added reversible components to left side
Parts:
- added B1: , E73:SW_TACT_ALPS_SKQGABE010, F.Cu at (209.2, 141.4)
- added TRRS1: TRRS-PJ-320A-dual, TRRS-PJ-320A-dual, F.Cu at (213.9, 116.8)
- moved D13 180.3 mm to (130.5, 163.8)
- moved D6 180.3 mm to (92.6, 152.8)
- moved S13 180.3 mm to (131.4, 158.9)
- moved S6 180.3 mm to (93.0, 147.8)
- moved D21 180.3 mm to (166.2, 178.9)
- moved S21 180.3 mm to (167.2, 174.0)
- moved D12 180.3 mm to (119.1, 109.7)
- moved D20 180.3 mm to (158.8, 117.3)
- moved D7 180.3 mm to (94.2, 133.9)
- moved D8 180.3 mm to (95.9, 114.9)
- moved S12 180.3 mm to (119.8, 104.7)
- moved S20 180.3 mm to (159.8, 112.4)
- moved S7 180.3 mm to (94.7, 128.9)
- moved S8 180.3 mm to (96.3, 110.0)
- moved D11 180.3 mm to (116.5, 128.5)
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Connections:
- D1 pad 1: (no net) -> P7
- D10 pad 1: (no net) -> P6
- D11 pad 1: (no net) -> P5
- D12 pad 1: (no net) -> P4
- D13 pad 1: (no net) -> P7
- D14 pad 1: (no net) -> P6
- D15 pad 1: (no net) -> P5
- D16 pad 1: (no net) -> P4
- D17 pad 1: (no net) -> P7
- D18 pad 1: (no net) -> P6
- D19 pad 1: (no net) -> P5
- D2 pad 1: (no net) -> P6
- D20 pad 1: (no net) -> P4
- D21 pad 1: (no net) -> P7
- D22 pad 1: (no net) -> P6
- D23 pad 1: (no net) -> P5
- D24 pad 1: (no net) -> P4
- D25 pad 1: (no net) -> P7
- D26 pad 1: (no net) -> P9
- D27 pad 1: (no net) -> P9
- D28 pad 1: (no net) -> P9
- D29 pad 1: (no net) -> P9
- D3 pad 1: (no net) -> P5
- D30 pad 1: (no net) -> P8
- D4 pad 1: (no net) -> P4
- D5 pad 1: (no net) -> P7
- D6 pad 1: (no net) -> P6
- D7 pad 1: (no net) -> P5
- D8 pad 1: (no net) -> P4
- D9 pad 1: (no net) -> P7
- S1 pad 1: (no net) -> P21
- S10 pad 1: (no net) -> P19
- S11 pad 1: (no net) -> P19
- S12 pad 1: (no net) -> P19
- S13 pad 1: (no net) -> P18
- S14 pad 1: (no net) -> P18
- S15 pad 1: (no net) -> P18
- S16 pad 1: (no net) -> P18
- S17 pad 1: (no net) -> P15
- S18 pad 1: (no net) -> P15
- S19 pad 1: (no net) -> P15
- S2 pad 1: (no net) -> P21
- S20 pad 1: (no net) -> P15
- S21 pad 1: (no net) -> P14
- S22 pad 1: (no net) -> P14
- S23 pad 1: (no net) -> P14
- S24 pad 1: (no net) -> P14
- S25 pad 1: (no net) -> P16
- S26 pad 1: (no net) -> P18
- S27 pad 1: (no net) -> P15
- S28 pad 1: (no net) -> P14
- S29 pad 1: (no net) -> P16
- S3 pad 1: (no net) -> P21
- S30 pad 1: (no net) -> P16
- S4 pad 1: (no net) -> P21
- S5 pad 1: (no net) -> P20
- S6 pad 1: (no net) -> P20
- S7 pad 1: (no net) -> P20
- S8 pad 1: (no net) -> P20
- S9 pad 1: (no net) -> P19
Other:
- outline, holes or cut-outs redrawn
