File: ergogen/pcbs/right.kicad_pcb (KiCad board)
At the start: 2 copper layers, 167 x 141 mm, 62 parts

Commit message: decided to go reversible pcb route, removed right side and added reversible components to left side
Parts:
- added B1: , E73:SW_TACT_ALPS_SKQGABE010, F.Cu at (264.5, 141.4)
- added TRRS1: TRRS-PJ-320A-dual, TRRS-PJ-320A-dual, F.Cu at (262.2, 116.4)
- moved D7 180.3 mm to (379.4, 133.9)
- moved D8 180.3 mm to (377.8, 114.9)
- moved S7 180.3 mm to (379.0, 128.9)
- moved S8 180.3 mm to (377.4, 110.0)
- moved D12 180.3 mm to (354.5, 109.7)
- moved D20 180.3 mm to (314.8, 117.3)
- moved S12 180.3 mm to (353.8, 104.7)
- moved S20 180.3 mm to (313.9, 112.4)
- moved D13 180.3 mm to (343.2, 163.8)
- moved D6 180.3 mm to (381.1, 152.8)
- moved S13 180.3 mm to (342.3, 158.9)
- moved S6 180.3 mm to (380.7, 147.8)
- moved D21 180.3 mm to (307.4, 178.9)
- moved S21 180.3 mm to (306.5, 174.0)
- moved D5 180.3 mm to (382.8, 171.7)
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Connections:
- D1 pad 1: (no net) -> P7
- D10 pad 1: (no net) -> P6
- D11 pad 1: (no net) -> P5
- D12 pad 1: (no net) -> P4
- D13 pad 1: (no net) -> P7
- D14 pad 1: (no net) -> P6
- D15 pad 1: (no net) -> P5
- D16 pad 1: (no net) -> P4
- D17 pad 1: (no net) -> P7
- D18 pad 1: (no net) -> P6
- D19 pad 1: (no net) -> P5
- D2 pad 1: (no net) -> P6
- D20 pad 1: (no net) -> P4
- D21 pad 1: (no net) -> P7
- D22 pad 1: (no net) -> P6
- D23 pad 1: (no net) -> P5
- D24 pad 1: (no net) -> P4
- D25 pad 1: (no net) -> P7
- D26 pad 1: (no net) -> P9
- D27 pad 1: (no net) -> P9
- D28 pad 1: (no net) -> P9
- D29 pad 1: (no net) -> P9
- D3 pad 1: (no net) -> P5
- D30 pad 1: (no net) -> P8
- D4 pad 1: (no net) -> P4
- D5 pad 1: (no net) -> P7
- D6 pad 1: (no net) -> P6
- D7 pad 1: (no net) -> P5
- D8 pad 1: (no net) -> P4
- D9 pad 1: (no net) -> P7
- MCU1 pad 10: P14 -> col_inner
- MCU1 pad 11: P16 -> col_inner2
- MCU1 pad 19: P4 -> row_upper
- MCU1 pad 20: P5 -> row_top
- MCU1 pad 21: P6 -> row_home
- MCU1 pad 22: P7 -> row_bottom
- MCU1 pad 23: P8 -> row_thumb2
- MCU1 pad 24: P9 -> row_thumb
- MCU1 pad 5: P21 -> col_pinky2
- MCU1 pad 6: P20 -> col_pinky
- MCU1 pad 7: P19 -> col_ring
- MCU1 pad 8: P18 -> col_middle
- MCU1 pad 9: P15 -> col_index
- S1 pad 1: (no net) -> P21
- S10 pad 1: (no net) -> P19
- S11 pad 1: (no net) -> P19
- S12 pad 1: (no net) -> P19
- S13 pad 1: (no net) -> P18
- S14 pad 1: (no net) -> P18
- S15 pad 1: (no net) -> P18
- S16 pad 1: (no net) -> P18
- S17 pad 1: (no net) -> P15
- S18 pad 1: (no net) -> P15
- S19 pad 1: (no net) -> P15
- S2 pad 1: (no net) -> P21
- S20 pad 1: (no net) -> P15
- S21 pad 1: (no net) -> P14
- S22 pad 1: (no net) -> P14
- S23 pad 1: (no net) -> P14
- S24 pad 1: (no net) -> P14
- S25 pad 1: (no net) -> P16
- S26 pad 1: (no net) -> P18
- S27 pad 1: (no net) -> P15
- S28 pad 1: (no net) -> P14
- S29 pad 1: (no net) -> P16
- S3 pad 1: (no net) -> P21
- S30 pad 1: (no net) -> P16
- S4 pad 1: (no net) -> P21
- S5 pad 1: (no net) -> P20
- S6 pad 1: (no net) -> P20
- S7 pad 1: (no net) -> P20
- S8 pad 1: (no net) -> P20
- S9 pad 1: (no net) -> P19
Other:
- outline, holes or cut-outs redrawn
